File: usbhub.kicad_sch (KiCad schematic)
At the start: 65 parts, among them IC1 FE1.1S, J1 USB_B, J2 USB-A, J3 USB-A, J4 USB-A, J5 USB-A, U1 USBLC6-2SC6, U2 24LC02, U3 USBLC6-2SC6, U4 USBLC6-2SC6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

Commit message: X7R -> X5R
Parts:
- C1, C12, C13, C14, C15: value 10 nF 2kV -> 10 nF
Other:
- note added: "0.1 uF caps X5R"
- note added: "10 uF caps X5R"
- note removed: "0.1 uF caps X7R"
- note removed: "10 uF caps X7R"
Changed lines of the file:
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@@
 		)
 	)
-	(text "0.1 uF caps X7R"
+	(text "0.1 uF caps X5R"
 		(exclude_from_sim no)
 		(at 252.476 63.754 0)
@@
 		)
 	)
-	(text "10 uF caps X7R\n"
+	(text "10 uF caps X5R\n"
 		(exclude_from_sim no)
 		(at 59.436 83.312 0)
@@
 			)
 		)
-		(property "Value" "10 nF 2kV"
+		(property "Value" "10 nF"
 			(at 235.204 148.59 90)
 			(show_name no)
@@
 			)
 		)
-		(property "Value" "10 nF 2kV"
+		(property "Value" "10 nF"
 			(at 241.808 116.84 90)
 			(show_name no)
@@
 			)
 		)
-		(property "Value" "10 nF 2kV"
-			(at 52.324 180.594 0)
+		(property "Value" "10 nF"
+			(at 47.752 181.356 0)
 			(show_name no)
 			(do_not_autoplace no)
@@
 			)
 		)
-		(property "Value" "10 nF 2kV"
+		(property "Value" "10 nF"
 			(at 241.554 88.9 90)
 			(show_name no)
@@
 			)
 		)
-		(property "Value" "10 nF 2kV"
-			(at 245.618 57.658 90)
+		(property "Value" "10 nF"
+			(at 240.792 57.658 90)
 			(show_name no)
 			(do_not_autoplace no)
